Commit message: structural refactoring, adding an earthquake generator

File: assignments/inverted_pendulum_optimal_control/models/inverted_pendulum/model.urdf (robot description, URDF)
Before this commit: robot inverted_pendulum, 4 links, 3 joints
Links:
- link base_link: geometry collision box size=5.0 0.5 0.1; visual box size=5.0 0.5 0.1
Joints:
- joint cart_to_base: limit lower=-2.0 upper=2.0 effort=1000.0 velocity=1000.0 -> lower=-2.5 upper=2.5 effort=1000.0 velocity=1000.0

Commit message: refactoring to motivate with earthquake cyber-physical twin science research needs

File: assignments/inverted_pendulum_optimal_control/models/inverted_pendulum/model.urdf (robot description, URDF)
Before this commit: robot inverted_pendulum, 4 links, 3 joints
Links:
- link base_link: geometry collision box size=5.0 0.2 0.1; visual box size=5.0 0.2 0.1
